File: Grid_PCB.kicad_pcb (KiCad board)
At the start: 2 copper layers, 223.2 x 22 mm, 42 parts, among them J1 Conn_01x04_Female, J10 LED_Conn, J11 Power_Conn, J2 Conn_01x04_Female, J3 Conn_01x04_Female, J4 Conn_01x04_Female, J5 Conn_01x04_Female, J6 Conn_01x04_Female, J7 Conn_01x04_Female, J8 Conn_01x04_Female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

Commit message: wave 4
Parts:
- removed the G*** at (154.3, 94.9)
- added G***: LOGO, grid:wave_pattern_4, F.Cu at (153.2, 100.0)
- added G***: LOGO, grid:wave_pattern_4, F.Cu at (162.5, 88.3)

Commit message: wave 4 skinny
Parts:
- removed the G*** at (153.2, 100.0)
- removed the G*** at (162.5, 88.3)
- added G***: LOGO, grid:wave_pattern_4_skinny, F.Cu at (162.0, 87.0)
- added G***: LOGO, grid:wave_pattern_4_skinny, F.Cu at (153.5, 102.1)

Commit message: wave fish
Parts:
- removed the G*** at (162.0, 87.0)
- removed the G*** at (153.5, 102.1)
- added G***: LOGO, grid:wave_fish, F.Cu at (224.0, 96.1)
- added G***: LOGO, grid:wave_fish, F.Cu at (153.6, 95.6)
- added G***: LOGO, grid:wave_fish, F.Cu at (82.8, 95.4)

Commit message: wave fish middle
Parts:
- removed the G*** at (224.0, 96.1)
- removed the G*** at (153.6, 95.6)
- added G***: LOGO, grid:wave_fish, F.Cu at (223.4, 92.2)
- added G***: LOGO, grid:wave_fish, F.Cu at (153.0, 91.7)
- moved G*** 3.92 mm to (82.2, 91.5)
Changed lines of the file:
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@@
   )
   (module grid:wave_fish (layer F.Cu)
-    (at 224.03308 96.08566)
+    (at 223.41332 92.21724)
     (fp_text reference G*** (at 0 0) (layer F.SilkS) hide
       (effects (font (size 1.524 1.524) (thickness 0.3)))
@@
   )
   (module grid:wave_fish (layer F.Cu)
-    (at 153.58872 95.5675)
+    (at 152.96896 91.69908)
     (fp_text reference G*** (at 0 0) (layer F.SilkS) hide
       (effects (font (size 1.524 1.524) (thickness 0.3)))
@@
   )
   (module grid:wave_fish (layer F.Cu)
-    (at 82.79638 95.39478)
+    (at 82.17662 91.52636)
     (fp_text reference G*** (at 0 0) (layer F.SilkS) hide
       (effects (font (size 1.524 1.524) (thickness 0.3)))

Commit message: wave fish thin, like this one the best
Parts:
- removed the G*** at (223.4, 92.2)
- removed the G*** at (153.0, 91.7)
- removed the G*** at (82.2, 91.5)
- added G***: LOGO, grid:wave_fish_small, F.Cu at (243.3, 86.9)
- added G***: LOGO, grid:wave_fish_small, F.Cu at (148.7, 101.5)
- added G***: LOGO, grid:wave_fish_small, F.Cu at (116.9, 101.5)
- added G***: LOGO, grid:wave_fish_small, F.Cu at (85.2, 101.5)
- added G***: LOGO, grid:wave_fish_small, F.Cu at (148.2, 86.9)
- added G***: LOGO, grid:wave_fish_small, F.Cu at (211.6, 86.9)
- added G***: LOGO, grid:wave_fish_small, F.Cu at (84.8, 86.9)
- added G***: LOGO, grid:wave_fish_small, F.Cu at (179.9, 86.9)
- added G***: LOGO, grid:wave_fish_small, F.Cu at (116.5, 86.9)
- added G***: LOGO, grid:wave_fish_small, F.Cu at (243.8, 101.5)
- added G***: LOGO, grid:wave_fish_small, F.Cu at (212.1, 101.5)
- added G***: LOGO, grid:wave_fish_small, F.Cu at (180.4, 101.5)
